File: io.kicad_sch (KiCad schematic)
At the start: 11 parts, among them J1 Conn_01x08, J10 Conn_01x02, J2 Conn_01x08, J4 USB_C_Receptacle_USB2.0_14P, J5 Conn_01x02, J6 Conn_01x02, J7 Conn_01x02, J8 Conn_01x02, J9 Conn_01x02

Commit message: Fix schematic review findings
Power:
- Input caps were in series with VIN; now VIN->GND, VIN tied to supply
- U4 (5V) runs from protected battery rail: 60V PTC, SS210 reverse-
  polarity diode, SMBJ43A TVS, 47uF/100V bulk; EN UVLO divider (30.3V/24.2V)
- U3 (3V3) cascaded from +5V so the MCU runs on USB power too
- TPS2116 power mux: buck has priority, USB VBUS fallback, no backfeed
- Output caps redesigned per TI Table 8-1 (LM6xx25 column); L2 -> 10uH
- U3 PG drives NRST (pulled to 3V3)
- Project LM656x5 symbol: EP numbered 21, PG/RT/MODE/VCC pin types fixed,
  limit text 65V (stock KiCad symbol had all of these wrong)
- New TI_RZT0020A footprint per TI land pattern 4228518/C

MCU / IO:
- GNDA tied to GND; HSE crystal uses 2-pin symbol; load caps 33pF
- USB data connected through hierarchy; VBUS separated from +5V,
  USBLC6 ESD, VBUS sense divider on PA9
- BOOT0 10k pull-down, R2 1k, latching slide switch; switch footprints
- TCAN330 decoupling, S/SHDN tied low, termination jumper JP1
- GPIO export: 100R series + SP0505 ESD; PTCs on exported 5V/3V3
- LED resistor/colour fixes; unused MCU pins marked no-connect
- Every BOM line has manufacturer, MPN and LCSC fields
- CAN/SPI netclasses defined; power nets removed from SPI class

Co-Authored-By: Claude Opus 5.5 <noreply@anthropic.com>
Parts:
- added C30: 4.7uF, Capacitor_SMD:C_0603_1608Metric, symbol Device:C
- added F2: 500mA, Fuse:Fuse_0805_2012Metric, symbol Device:Polyfuse_Small
- added F3: 350mA, Fuse:Fuse_0805_2012Metric, symbol Device:Polyfuse_Small
- added R19, R20, R21, R22, R23: 100R, Resistor_SMD:R_0402_1005Metric, symbol Device:R_Small
- added U6: USBLC6-2SC6, Package_TO_SOT_SMD:SOT-23-6, symbol Power_Protection:USBLC6-2SC6
- added U7: SP0505BAHT, Package_TO_SOT_SMD:SOT-23-6, symbol Power_Protection:SP0505BAHT
- J1, J2: value Conn_01x08 -> Micro-Fit 1x08; Manufacturer (none) -> Molex; Manufacturer Part Number (none) -> 0436500800
- J10, J5, J6, J7, J8, J9: value Conn_01x02 -> Micro-Fit 1x02; Manufacturer (none) -> Molex; Manufacturer Part Number (none) -> 0436500200
- J4: value USB_C_Receptacle_USB2.0_14P -> USB4105-GF-A; LCSC Part Number (none) -> C3020560; Manufacturer (none) -> GCT; Manufacturer Part Number (none) -> USB4105-GF-A
- R14, R15: LCSC Part Number (none) -> C25905; Manufacturer (none) -> UNI-ROYAL; Manufacturer Part Number (none) -> 0402WGF5101TCE
Connections:
- net +3V3: now also F3.1; no longer J2.2 (Pin_2)
- net +5V: now also F2.1; no longer J10.1 (Pin_1), J2.1 (Pin_1), J4.A4 (VBUS), J4.A9 (VBUS), J4.B4 (VBUS), J4.B9 (VBUS)
- net GND: now also C30.2, U6.2 (GND), U7.2 (A)
- net GPIO0: now also R19.1; no longer J2.3 (Pin_3)
- net GPIO1: now also R20.1; no longer J2.4 (Pin_4)
- net GPIO2: now also R21.1; no longer J2.5 (Pin_5)
- net GPIO3: now also R22.1; no longer J2.6 (Pin_6)
- net GPIO4: now also R23.1; no longer J2.7 (Pin_7)
- net USB.DM: now also U6.3 (I/O2), U6.4 (I/O2)
- net USB.DP: now also U6.1 (I/O1), U6.6 (I/O1)
- new net +3V3_EXT: F3.2, J2.2 (Pin_2)
- new net +5V_EXT: F2.2, J10.1 (Pin_1), J2.1 (Pin_1)
- new net EXT0: J2.3 (Pin_3), R19.2, U7.1 (K)
- new net EXT1: J2.4 (Pin_4), R20.2, U7.3 (K)
- new net EXT2: J2.5 (Pin_5), R21.2, U7.4 (K)
- new net EXT3: J2.6 (Pin_6), R22.2, U7.5 (K)
- new net EXT4: J2.7 (Pin_7), R23.2, U7.6 (K)
- new net VBUS: C30.1, J4.A4 (VBUS), J4.A9 (VBUS), J4.B4 (VBUS), J4.B9 (VBUS), U6.5 (VBUS)
Other:
- note added: "EXPORTED RAIL PROTECTION"
- note added: "GPIO ESD PA4 is 3.3V-only (TTa)!"
- note added: "R19-R23 100R GPIO series"
- note added: "USB ESD + VBUS"

Commit message: Update PCB and schematics after review fixes
Co-Authored-By: Claude Opus 5.5 <noreply@anthropic.com>
Other:
- moved on the sheet: F2, F3
