File: mcu.kicad_sch (KiCad schematic)
At the start: 2 parts, among them U1 STM32F405RGTx

Commit message: progress checkin
Parts:
- added U2: TCAN330, Package_SO:SOIC-8_3.9x4.9mm_P1.27mm, symbol Interface_CAN_LIN:TCAN330
Connections:
- net +3V3: now also U2.3 (VCC)
- net CAN_RX: now also U2.4 (RXD)
- net CAN_TX: now also U2.1 (TXD)
- net GND: now also U2.2 (GND)
- new net CAN_H: U2.7 (CANH)
- new net CAN_L: U2.6 (CANL)
- no-connect marks 1 -> 3
Other:
- note added: "CAN"
- moved on the sheet: C1, U1

Commit message: syncing
Parts:
- added C10, C27, C28, C9: 2.2uF, symbol Device:C
- added C11, C12, C13, C14, C15, C16: 100nf, symbol Device:C
- added C17: 1uF, symbol Device:C
- added C18, C19: 15pF, symbol Device:C
- added D1: RED, symbol Device:LED
- added D2: GREEN, symbol Device:LED
- added D3: BLUE, symbol Device:LED
- added J3: Tag Connect, Connector:Tag-Connect_TC2030-IDC-FP_2x03_P1.27mm_Vertical, symbol Connector:Conn_ARM_SWD_TagConnect_TC2030
- added R10: 1k, symbol Device:R
- added R11, R9: 220R, symbol Device:R
- added R13: 10k, symbol Device:R
- added R2: 100k, symbol Device:R
- added R3, R4, R6, R7: 0R, symbol Device:R
- added R5: 0R, Resistor_SMD:R_0402_1005Metric, symbol Device:R
- added R8: 120R, symbol Device:R
- added SW1: SW_Push, symbol Switch:SW_Push
- added SW2: SW_Push_SPDT, symbol Switch:SW_Push_SPDT
- added Y2: Crystal_GND2_Small, symbol Device:Crystal_GND2_Small
Connections:
- net +3V3: now also U1.1 (VBAT), C12.1, C13.1, C14.1, C15.1, C16.1, C17.1, C27.2, C28.2, J3.1 (VCC), SW2.3 (C)
- net CAN_H: now also R8.1
- net CAN_L: now also R8.2
- net CAN_RX: now also R3.2, R6.1; no longer U1.45 (PA12)
- net CAN_TX: now also R4.2, R7.1; no longer U1.44 (PA11)
- net GND: now also C10.1, C11.2, C12.2, C13.2, C14.2, C15.2, C16.2, C17.2, C18.1, C19.2, C9.1, D1.1 (K), D2.1 (K), D3.1 (K), J3.5 (GND), R13.1, SW1.1, SW2.1 (A), Y2.2; no longer U1.12 (VSSA)
- net at U1.10 (PC2): now also R10.2
- net GPIO0: now reaches U1.14 (PA0)
- net GPIO1: now reaches U1.15 (PA1)
- net GPIO2: now reaches U1.16 (PA2)
- net GPIO3: now reaches U1.17 (PA3)
- net GPIO4: now reaches U1.20 (PA4)
- net at U1.28 (PB2): now also R13.2
- net display.SCK: now reaches U1.29 (PB10)
- net display.DC: now reaches U1.30 (PB11)
- net at U1.31 (VCAP_1): now also C9.2
- net display.CS: now reaches U1.33 (PB12)
- net display.RES: now reaches U1.34 (PB13)
- net display.SDA(MOSI): now reaches U1.36 (PB15)
- net SWDIO: now reaches U1.46 (PA13)
- net SWDIO: now also J3.2 (SWDIO)
- net at U1.47 (VCAP_2): now also C10.2
- net SWCLK: now reaches U1.49 (PA14)
- net SWCLK: now also J3.4 (SWCLK)
- net OSC32_IN: now reaches U1.5 (PH0)
- net OSC32_IN: now also C18.2, Y2.1
- net SWO: now reaches U1.55 (PB3)
- net SWO: now also J3.6 (SWO)
- net OSC32_OUT: now reaches U1.6 (PH1)
- net OSC32_OUT: now also R5.1
- net at U1.60 (BOOT0): now also R2.2
- net at U1.61 (PB8): now also R3.1, R7.2
- net at U1.62 (PB9): now also R4.1, R6.2
- net NRST: now reaches U1.7 (NRST)
- net NRST: now also C11.1, J3.3 (~{RESET}), SW1.2
- net at U1.8 (PC0): now also R11.2
- net at U1.9 (PC1): now also R9.2
- new net: D2.2 (A), R9.1
- new net: R2.1, SW2.2 (B)
- new net: D1.2 (A), R11.1
- new net: C19.1, R5.2, Y2.3
- new net: D3.2 (A), R10.1
- new net GNDA: C27.1, C28.1, U1.12 (VSSA)
- new net USB.DM: U1.44 (PA11)
- new net USB.DP: U1.45 (PA12)
- no-connect marks 3 -> 2
Other:
- note added: "CRYSTAL"
- note added: "NRST"
- note added: "TAG CONNECT"
- note added: "VDD DECOUPLING"
- moved on the sheet: C1, U1, U2

Commit message: assigning footprints
Parts:
- C1, C10, C11, C12, C13, C14, C15, C16, C17, C18, C19, C27, C28, C9: footprint (none) -> Capacitor_SMD:C_0402_1005Metric
- D1, D2, D3: footprint (none) -> LED_SMD:LED_0603_1608Metric
- R10, R11, R13, R2, R8, R9: footprint (none) -> Resistor_SMD:R_0402_1005Metric
- R3, R4, R6, R7: footprint (none) -> Resistor_SMD:R_0603_1608Metric
- R5: footprint Resistor_SMD:R_0402_1005Metric -> Resistor_SMD:R_0603_1608Metric
- Y2: footprint (none) -> Crystal:Crystal_SMD_5032-2Pin_5.0x3.2mm
Changed lines of the file:
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@@
 			(justify left)
 		)
-		(property "Net Class" "SPI"
+		(property "Netclass" "SPI"
 			(at 244.348 152.146 0)
 			(show_name no)
@@
 			(justify left)
 		)
-		(property "Net Class" "CAN"
+		(property "Netclass" "CAN"
 			(at 74.93 168.91 0)
 			(show_name no)
@@
 			)
 		)
-		(property "Footprint" ""
+		(property "Footprint" "LED_SMD:LED_0603_1608Metric"
 			(at 125.73 87.63 0)
 			(hide yes)
@@
 			)
 		)
-		(property "Footprint" ""
+		(property "Footprint" "Resistor_SMD:R_0402_1005Metric"
 			(at 120.65 69.088 90)
 			(hide yes)
@@
 			)
 		)
-		(property "Footprint" ""
+		(property "Footprint" "Resistor_SMD:R_0603_1608Metric"
 			(at 255.27 134.112 90)
 			(hide yes)
@@
 			)
 		)
-		(property "Footprint" ""
+		(property "Footprint" "Capacitor_SMD:C_0402_1005Metric"
 			(at 171.7548 153.67 0)
 			(hide yes)
@@
 			)
 		)
-		(property "Footprint" ""
+		(property "Footprint" "Capacitor_SMD:C_0402_1005Metric"
 			(at 30.1752 35.56 0)
 			(hide yes)
@@
 			)
 		)
-		(property "Footprint" ""
+		(property "Footprint" "Capacitor_SMD:C_0402_1005Metric"
 			(at 55.5752 35.56 0)
 			(hide yes)
@@
 			)
 		)
-		(property "Footprint" ""
+		(property "Footprint" "LED_SMD:LED_0603_1608Metric"
 			(at 125.73 81.28 0)
 			(hide yes)
@@
 			)
 		)
-		(property "Footprint" ""
+		(property "Footprint" "Capacitor_SMD:C_0402_1005Metric"
 			(at 122.2248 130.81 0)
 			(hide yes)
@@
 			)
 		)
-		(property "Footprint" ""
+		(property "Footprint" "Capacitor_SMD:C_0402_1005Metric"
 			(at 68.2752 35.56 0)
 			(hide yes)
@@
 			)
 		)
-		(property "Footprint" ""
+		(property "Footprint" "Capacitor_SMD:C_0402_1005Metric"
 			(at 106.3752 35.56 0)
 			(hide yes)
@@
 			)
 		)
-		(property "Footprint" ""
+		(property "Footprint" "Resistor_SMD:R_0603_1608Metric"
 			(at 255.27 116.332 90)
 			(hide yes)
@@
 			)
 		)
-		(property "Footprint" ""
+		(property "Footprint" "Capacitor_SMD:C_0402_1005Metric"
 			(at 91.1352 35.56 0)
 			(hide yes)
@@
 			)
 		)
-		(property "Footprint" ""
+		(property "Footprint" "Capacitor_SMD:C_0402_1005Metric"
 			(at 137.4648 130.81 0)
 			(hide yes)
@@
 			)
 		)
-		(property "Footprint" ""
+		(property "Footprint" "Capacitor_SMD:C_0402_1005Metric"
 			(at 42.8752 35.56 0)
 			(hide yes)
@@
 			)
 		)
-		(property "Footprint" ""
+		(property "Footprint" "Capacitor_SMD:C_0402_1005Metric"
 			(at 33.02 91.7448 0)
 			(hide yes)
@@
 			)
 		)
-		(property "Footprint" ""
+		(property "Footprint" "Crystal:Crystal_SMD_5032-2Pin_5.0x3.2mm"
 			(at 45.72 92.71 0)
 			(hide yes)
@@
 			)
 		)
-		(property "Footprint" ""
+		(property "Footprint" "Resistor_SMD:R_0402_1005Metric"
 			(at 133.35 83.058 90)
 			(hide yes)
@@
 			)
 		)
-		(property "Footprint" ""
+		(property "Footprint" "Resistor_SMD:R_0402_1005Metric"
 			(at 51.562 173.99 90)
 			(hide yes)
@@
 			)
 		)
-		(property "Footprint" "Resistor_SMD:R_0402_1005Metric"
+		(property "Footprint" "Resistor_SMD:R_0603_1608Metric"
 			(at 51.562 86.36 90)
 			(hide yes)
@@
 			)
 		)
-		(property "Footprint" ""
+		(property "Footprint" "Resistor_SMD:R_0603_1608Metric"
 			(at 255.27 132.588 90)
 			(hide yes)
@@
 			)
 		)
-		(property "Footprint" ""
+		(property "Footprint" "Capacitor_SMD:C_0402_1005Metric"
 			(at 18.7452 35.56 0)
 			(hide yes)
@@
 			)
 		)
-		(property "Footprint" ""
+		(property "Footprint" "Resistor_SMD:R_0402_1005Metric"
 			(at 133.35 95.758 90)
 			(hide yes)
@@
 			)
 		)
-		(property "Footprint" ""
+		(property "Footprint" "Resistor_SMD:R_0402_1005Metric"
 			(at 204.978 114.3 90)
 			(hide yes)
@@
 			)
 		)
-		(property "Footprint" ""
+		(property "Footprint" "Capacitor_SMD:C_0402_1005Metric"
 			(at 184.4548 153.67 0)
 			(hide yes)
@@
 			)
 		)
-		(property "Footprint" ""
+		(property "Footprint" "Resistor_SMD:R_0402_1005Metric"
 			(at 133.35 89.408 90)
 			(hide yes)
@@
 			)
 		)
-		(property "Footprint" ""
+		(property "Footprint" "Capacitor_SMD:C_0402_1005Metric"
 			(at 39.0652 59.69 0)
 			(hide yes)
@@
 			)
 		)
-		(property "Footprint" ""
+		(property "Footprint" "LED_SMD:LED_0603_1608Metric"
 			(at 125.73 93.98 0)
 			(hide yes)
@@
 			)
 		)
-		(property "Footprint" ""
+		(property "Footprint" "Capacitor_SMD:C_0402_1005Metric"
 			(at 64.77 91.7448 0)
 			(hide yes)
@@
 			)
 		)
-		(property "Footprint" ""
+		(property "Footprint" "Resistor_SMD:R_0603_1608Metric"
 			(at 255.27 124.968 90)
 			(hide yes)
