File: mcu.kicad_sch (KiCad schematic)
At the start: 34 parts, among them J3 Tag Connect, SW1 SW_Push, SW2 SW_Push_SPDT, U1 STM32F405RGTx, U2 TCAN330, Y2 Crystal_GND2_Small

Commit message: Fix schematic review findings
Power:
- Input caps were in series with VIN; now VIN->GND, VIN tied to supply
- U4 (5V) runs from protected battery rail: 60V PTC, SS210 reverse-
  polarity diode, SMBJ43A TVS, 47uF/100V bulk; EN UVLO divider (30.3V/24.2V)
- U3 (3V3) cascaded from +5V so the MCU runs on USB power too
- TPS2116 power mux: buck has priority, USB VBUS fallback, no backfeed
- Output caps redesigned per TI Table 8-1 (LM6xx25 column); L2 -> 10uH
- U3 PG drives NRST (pulled to 3V3)
- Project LM656x5 symbol: EP numbered 21, PG/RT/MODE/VCC pin types fixed,
  limit text 65V (stock KiCad symbol had all of these wrong)
- New TI_RZT0020A footprint per TI land pattern 4228518/C

MCU / IO:
- GNDA tied to GND; HSE crystal uses 2-pin symbol; load caps 33pF
- USB data connected through hierarchy; VBUS separated from +5V,
  USBLC6 ESD, VBUS sense divider on PA9
- BOOT0 10k pull-down, R2 1k, latching slide switch; switch footprints
- TCAN330 decoupling, S/SHDN tied low, termination jumper JP1
- GPIO export: 100R series + SP0505 ESD; PTCs on exported 5V/3V3
- LED resistor/colour fixes; unused MCU pins marked no-connect
- Every BOM line has manufacturer, MPN and LCSC fields
- CAN/SPI netclasses defined; power nets removed from SPI class

Co-Authored-By: Claude Opus 5.5 <noreply@anthropic.com>
Parts:
- added C29: 100nF, Capacitor_SMD:C_0402_1005Metric, symbol Device:C
- added JP1: TERM, Jumper:SolderJumper-2_P1.3mm_Bridged_RoundedPad1.0x1.5mm, symbol Jumper:SolderJumper_2_Bridged
- added R16: 10k, Resistor_SMD:R_0402_1005Metric, symbol Device:R
- added R17: 22k, Resistor_SMD:R_0402_1005Metric, symbol Device:R
- added R18: 33k, Resistor_SMD:R_0402_1005Metric, symbol Device:R
- C1: footprint Capacitor_SMD:C_0402_1005Metric -> Capacitor_SMD:C_0805_2012Metric; LCSC Part Number (none) -> C15850; Manufacturer (none) -> Samsung; Manufacturer Part Number (none) -> CL21A106KAYNNNE
- C10, C27, C28, C9: LCSC Part Number (none) -> C12530; Manufacturer (none) -> Samsung; Manufacturer Part Number (none) -> CL05A225MQ5NSNC
- C11, C12, C13, C14, C15, C16: value 100nf -> 100nF; LCSC Part Number (none) -> C307331; Manufacturer (none) -> Samsung; Manufacturer Part Number (none) -> CL05B104KB54PNC
- C17: LCSC Part Number (none) -> C52923; Manufacturer (none) -> Samsung; Manufacturer Part Number (none) -> CL05A105KA5NQNC
- C18, C19: value 15pF -> 33pF; LCSC Part Number C1644 -> C1562; Manufacturer (none) -> FH; Manufacturer Part Number (none) -> 0402CG330J500NT
- D1: LCSC Part Number (none) -> C2286; Manufacturer (none) -> KENTO; Manufacturer Part Number (none) -> KT-0603R
- D2: value GREEN -> Y-GRN; LCSC Part Number (none) -> C2289; Manufacturer (none) -> KENTO; Manufacturer Part Number (none) -> KT-0603YG
- D3: LCSC Part Number (none) -> C2986058; Manufacturer (none) -> Everlight; Manufacturer Part Number (none) -> 19-217/BHC-ZL1M2RY/6T
- R10: value 1k -> 68R; LCSC Part Number (none) -> C2909380; Manufacturer (none) -> FOJAN; Manufacturer Part Number (none) -> FRC0402F68R0TS
- R11, R9: LCSC Part Number (none) -> C25091; Manufacturer (none) -> UNI-ROYAL; Manufacturer Part Number (none) -> 0402WGF2200TCE
- R13: LCSC Part Number (none) -> C25744; Manufacturer (none) -> UNI-ROYAL; Manufacturer Part Number (none) -> 0402WGF1002TCE
- R2: value 100k -> 1k; LCSC Part Number (none) -> C11702; Manufacturer (none) -> UNI-ROYAL; Manufacturer Part Number (none) -> 0402WGF1001TCE
- R3, R4, R5, R6, R7: LCSC Part Number (none) -> C21189; Manufacturer (none) -> UNI-ROYAL; Manufacturer Part Number (none) -> 0603WAF0000T5E
- R8: LCSC Part Number (none) -> C25079; Manufacturer (none) -> UNI-ROYAL; Manufacturer Part Number (none) -> 0402WGF1200TCE
- SW1: value SW_Push -> RESET; footprint (none) -> Button_Switch_SMD:SW_Push_1P1T_XKB_TS-1187A; LCSC Part Number (none) -> C318884; Manufacturer (none) -> XKB; Manufacturer Part Number (none) -> TS-1187A-B-A-B
- SW2: value SW_Push_SPDT -> BOOT0; footprint (none) -> Button_Switch_SMD:SW_SPDT_Shouhan_MSK12C02; symbol Switch:SW_Push_SPDT -> Switch:SW_SPDT; LCSC Part Number (none) -> C431540; Manufacturer (none) -> SHOU HAN; Manufacturer Part Number (none) -> MSK12C02
- U1: value STM32F405RGTx -> STM32F405RGT6; LCSC Part Number (none) -> C15742; Manufacturer (none) -> ST; Manufacturer Part Number (none) -> STM32F405RGT6
- U2: value TCAN330 -> TCAN330DR; LCSC Part Number (none) -> C2652876; Manufacturer (none) -> TI; Manufacturer Part Number (none) -> TCAN330DR
- Y2: value Crystal_GND2_Small -> 8MHz 20pF; symbol Device:Crystal_GND2_Small -> Device:Crystal_Small; Manufacturer (none) -> YXC; Manufacturer Part Number (none) -> X50328MSB2GI
Connections:
- net GNDA is gone; now on net GND: C27.1, C28.1, U1.12 (VSSA)
- net +3V3: now also C29.1
- net CAN_L: now also JP1.1 (A); no longer R8.2
- net GND: now also U2.5 (SHDN), U2.8 (S), C29.2, R16.2, R18.2; no longer Y2.2
- net at R2.2, U1.60 (BOOT0): now also R16.1
- net at C19.1, R5.2: now also Y2.2; no longer Y2.3
- net VBUS_SENSE: now reaches U1.42 (PA9)
- net VBUS_SENSE: now also R17.2, R18.1
- net OSC32_IN renamed HSE_IN
- net OSC32_OUT renamed HSE_OUT
- new net: JP1.2 (B), R8.2
- new net VBUS: R17.1
- no-connect marks 2 -> 27
Other:
- note added: "USB VBUS DETECT 5V -> 3.0V on PA9"
