File: power.kicad_sch (KiCad schematic)
At the start: 1 part

Commit message: progress checkin
Other:
- moved on the sheet: U3

Commit message: syncing
Parts:
- added C2, C24: 0.1uF, symbol Device:C
- added C20, C21, C3, C4: 4.7uF, symbol Device:C
- added C22, C23, C5, C6: 100nF, symbol Device:C
- added C25, C8: 1uF, symbol Device:C
- added C26: 55uF, symbol Device:C
- added C7: 94uF, symbol Device:C
- added L1: 6.8uH, symbol Device:L
- added L2: 8.2uH, symbol Device:L
- added R1, R12: R, symbol Device:R
- added U4: LM65625SRZTR, symbol Converter_DCDC:LM656x5
- U3: value (none) -> LM65625SRZTR
Connections:
- net GND: now reaches U3. (GND)
- net GND: now also U3.19 (PGND2), U3.3 (FB), U3.5 (MODE/SYNC), U3.9 (PGND1), C25.2, C26.2, C7.2, C8.2, U4. (GND), U4.19 (PGND2), U4.5 (MODE/SYNC), U4.9 (PGND1)
- net at U3.11 (VIN1): now also U3.17 (VIN2), U3.7 (EN/UVLO), C3.2, C4.2, C5.2, C6.2
- net at U3.13 (SW1): now also U3.14 (SW2), C2.2, L1.1
- net at U3.15 (BOOT): now also C2.1
- net at U3.2 (PG): now also R1.2
- net +3V3: now reaches U3.20 (BIAS)
- net +3V3: now also C7.1, L1.2
- net LM656_3V3_VCC: now reaches U3.4 (VCC)
- net LM656_3V3_VCC: now also U3.6 (RT), C8.1, R1.1
- new net: C24.1, U4.15 (BOOT)
- new net: C24.2, L2.1, U4.13 (SW1), U4.14 (SW2)
- new net: C20.2, C21.2, C22.2, C23.2, U4.11 (VIN1), U4.17 (VIN2), U4.7 (EN/UVLO)
- new net: R12.2, U4.2 (PG)
- new net +5V: C26.1, L2.2, U4.20 (BIAS)
- new net LM656_5V_VCC: C25.1, R12.1, U4.3 (FB), U4.4 (VCC), U4.6 (RT)
- new net VCC: C20.1, C21.1, C22.1, C23.1, C3.1, C4.1, C5.1, C6.1
Other:
- note added: "3V3 REG"
- note added: "5V REG"
- moved on the sheet: U3

Commit message: assigning footprints
Parts:
- C2, C20, C21, C22, C23, C24, C25, C26, C3, C4, C5, C6, C7, C8: footprint (none) -> Capacitor_SMD:C_0402_1005Metric
- R1, R12: value R -> 100k; footprint (none) -> Resistor_SMD:R_0402_1005Metric
- U3, U4: footprint (none) -> Jackson:RZT0020A-MFG
Changed lines of the file:
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@@
 			)
 		)
-		(property "Footprint" ""
+		(property "Footprint" "Capacitor_SMD:C_0402_1005Metric"
 			(at 235.9152 72.39 0)
 			(hide yes)
@@
 			)
 		)
-		(property "Footprint" ""
+		(property "Footprint" "Capacitor_SMD:C_0402_1005Metric"
 			(at 102.87 53.6448 0)
 			(hide yes)
@@
 			)
 		)
-		(property "Footprint" ""
+		(property "Footprint" "Capacitor_SMD:C_0402_1005Metric"
 			(at 238.76 53.6448 0)
 			(hide yes)
@@
 			)
 		)
-		(property "Footprint" ""
+		(property "Footprint" "Jackson:RZT0020A-MFG"
 			(at 76.2 57.15 0)
 			(hide yes)
@@
 		)
 		(property "Field5" ""
+			(at 76.2 57.15 0)
+			(hide yes)
+			(show_name no)
+			(do_not_autoplace no)
+			(effects
+				(font
+					(size 1.27 1.27)
+				)
+			)
+		)
+		(property "LCSC Part Number" ""
+			(at 76.2 57.15 0)
+			(hide yes)
+			(show_name no)
+			(do_not_autoplace no)
+			(effects
+				(font
+					(size 1.27 1.27)
+				)
+			)
+		)
+		(property "Manufacturer" ""
+			(at 76.2 57.15 0)
+			(hide yes)
+			(show_name no)
+			(do_not_autoplace no)
+			(effects
+				(font
+					(size 1.27 1.27)
+				)
+			)
+		)
+		(property "Mouser Part Number" ""
+			(at 76.2 57.15 0)
+			(hide yes)
+			(show_name no)
+			(do_not_autoplace no)
+			(effects
+				(font
+					(size 1.27 1.27)
+				)
+			)
+		)
+		(property "Digikey Part Number" ""
+			(at 76.2 57.15 0)
+			(hide yes)
+			(show_name no)
+			(do_not_autoplace no)
+			(effects
+				(font
+					(size 1.27 1.27)
+				)
+			)
+		)
+		(property "Manufacturer Part Number" ""
 			(at 76.2 57.15 0)
 			(hide yes)
@@
 			)
 		)
-		(property "Footprint" ""
+		(property "Footprint" "Capacitor_SMD:C_0402_1005Metric"
 			(at 54.3052 39.37 0)
 			(hide yes)
@@
 			)
 		)
-		(property "Footprint" ""
+		(property "Footprint" "Capacitor_SMD:C_0402_1005Metric"
 			(at 190.1952 39.37 0)
 			(hide yes)
@@
 		(fields_autoplaced yes)
 		(property "Reference" "R1"
-			(at 36.83 69.8499 0)
+			(at 36.83 69.85 0)
 			(show_name no)
 			(do_not_autoplace no)
@@
 			)
 		)
-		(property "Value" "R"
-			(at 36.83 72.3899 0)
+		(property "Value" "100k"
+			(at 36.83 72.39 0)
 			(show_name no)
 			(do_not_autoplace no)
@@
 			)
 		)
-		(property "Footprint" ""
+		(property "Footprint" "Resistor_SMD:R_0402_1005Metric"
 			(at 32.512 71.12 90)
 			(hide yes)
@@
 			)
 		)
-		(property "Footprint" ""
+		(property "Footprint" "Capacitor_SMD:C_0402_1005Metric"
 			(at 67.0052 39.37 0)
 			(hide yes)
@@
 			)
 		)
-		(property "Footprint" ""
+		(property "Footprint" "Capacitor_SMD:C_0402_1005Metric"
 			(at 202.8952 39.37 0)
 			(hide yes)
@@
 			)
 		)
-		(property "Footprint" ""
+		(property "Footprint" "Capacitor_SMD:C_0402_1005Metric"
 			(at 100.0252 72.39 0)
 			(hide yes)
@@
 			)
 		)
-		(property "Footprint" ""
+		(property "Footprint" "Jackson:RZT0020A-MFG"
 			(at 212.09 57.15 0)
 			(hide yes)
@@
 			)
 		)
-		(property "Footprint" ""
+		(property "Footprint" "Capacitor_SMD:C_0402_1005Metric"
 			(at 28.9052 39.37 0)
 			(hide yes)
@@
 			)
 		)
-		(property "Footprint" ""
+		(property "Footprint" "Capacitor_SMD:C_0402_1005Metric"
 			(at 41.6052 39.37 0)
 			(hide yes)
@@
 			)
 		)
-		(property "Footprint" ""
+		(property "Footprint" "Capacitor_SMD:C_0402_1005Metric"
 			(at 164.7952 39.37 0)
 			(hide yes)
@@
 			)
 		)
-		(property "Footprint" ""
+		(property "Footprint" "Capacitor_SMD:C_0402_1005Metric"
 			(at 120.3452 54.61 0)
 			(hide yes)
@@
 			)
 		)
-		(property "Footprint" ""
+		(property "Footprint" "Capacitor_SMD:C_0402_1005Metric"
 			(at 256.2352 54.61 0)
 			(hide yes)
@@
 			)
 		)
-		(property "Value" "R"
+		(property "Value" "100k"
 			(at 172.72 72.3899 0)
 			(show_name no)
@@
 			)
 		)
-		(property "Footprint" ""
+		(property "Footprint" "Resistor_SMD:R_0402_1005Metric"
 			(at 168.402 71.12 90)
 			(hide yes)
@@
 		)
 		(property "Description" "Resistor"
+			(at 170.18 71.12 0)
+			(hide yes)
+			(show_name no)
+			(do_not_autoplace no)
+			(effects
+				(font
+					(size 1.27 1.27)
+				)
+			)
+		)
+		(property "LCSC Part Number" ""
+			(at 170.18 71.12 0)
+			(hide yes)
+			(show_name no)
+			(do_not_autoplace no)
+			(effects
+				(font
+					(size 1.27 1.27)
+				)
+			)
+		)
+		(property "Manufacturer" ""
+			(at 170.18 71.12 0)
+			(hide yes)
+			(show_name no)
+			(do_not_autoplace no)
+			(effects
+				(font
+					(size 1.27 1.27)
+				)
+			)
+		)
+		(property "Mouser Part Number" ""
+			(at 170.18 71.12 0)
+			(hide yes)
+			(show_name no)
+			(do_not_autoplace no)
+			(effects
+				(font
+					(size 1.27 1.27)
+				)
+			)
+		)
+		(property "Digikey Part Number" ""
+			(at 170.18 71.12 0)
+			(hide yes)
+			(show_name no)
+			(do_not_autoplace no)
+			(effects
+				(font
+					(size 1.27 1.27)
+				)
+			)
+		)
+		(property "Manufacturer Part Number" ""
 			(at 170.18 71.12 0)
 			(hide yes)
@@
 			)
 		)
-		(property "Footprint" ""
+		(property "Footprint" "Capacitor_SMD:C_0402_1005Metric"
 			(at 177.4952 39.37 0)
 			(hide yes)
