File: power.kicad_sch (KiCad schematic)
At the start: 20 parts, among them U3 LM65625SRZTR, U4 LM65625SRZTR

Commit message: Snapshot before schematic review fixes
Co-Authored-By: Claude Opus 5.5 <noreply@anthropic.com>
Parts:
- L1: footprint (none) -> jackson:Inductor_SMD_7.4mmx6.6mm; LCSC Part Number (none) -> C51933839
- L2: footprint (none) -> jackson:Inductor_SMD_7.4mmx6.6mm; LCSC Part Number (none) -> C53462990
Changed lines of the file:
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@@
 			)
 		)
-		(property "Footprint" ""
+		(property "Footprint" "jackson:Inductor_SMD_7.4mmx6.6mm"
 			(at 243.84 46.99 0)
 			(hide yes)
@@
 		)
 		(property "Description" "Inductor"
+			(at 243.84 46.99 0)
+			(hide yes)
+			(show_name no)
+			(do_not_autoplace no)
+			(effects
+				(font
+					(size 1.27 1.27)
+				)
+			)
+		)
+		(property "LCSC Part Number" "C53462990"
 			(at 243.84 46.99 0)
 			(hide yes)
@@
 			)
 		)
-		(property "Footprint" ""
+		(property "Footprint" "jackson:Inductor_SMD_7.4mmx6.6mm"
 			(at 107.95 46.99 0)
 			(hide yes)
@@
 			(at 107.95 46.99 0)
 			(hide yes)
+			(show_name no)
+			(do_not_autoplace no)
+			(effects
+				(font
+					(size 1.27 1.27)
+				)
+			)
+		)
+		(property "LCSC Part Number" "C51933839"
+			(at 107.95 46.99 0)
+			(hide yes)

Commit message: Fix schematic review findings
Power:
- Input caps were in series with VIN; now VIN->GND, VIN tied to supply
- U4 (5V) runs from protected battery rail: 60V PTC, SS210 reverse-
  polarity diode, SMBJ43A TVS, 47uF/100V bulk; EN UVLO divider (30.3V/24.2V)
- U3 (3V3) cascaded from +5V so the MCU runs on USB power too
- TPS2116 power mux: buck has priority, USB VBUS fallback, no backfeed
- Output caps redesigned per TI Table 8-1 (LM6xx25 column); L2 -> 10uH
- U3 PG drives NRST (pulled to 3V3)
- Project LM656x5 symbol: EP numbered 21, PG/RT/MODE/VCC pin types fixed,
  limit text 65V (stock KiCad symbol had all of these wrong)
- New TI_RZT0020A footprint per TI land pattern 4228518/C

MCU / IO:
- GNDA tied to GND; HSE crystal uses 2-pin symbol; load caps 33pF
- USB data connected through hierarchy; VBUS separated from +5V,
  USBLC6 ESD, VBUS sense divider on PA9
- BOOT0 10k pull-down, R2 1k, latching slide switch; switch footprints
- TCAN330 decoupling, S/SHDN tied low, termination jumper JP1
- GPIO export: 100R series + SP0505 ESD; PTCs on exported 5V/3V3
- LED resistor/colour fixes; unused MCU pins marked no-connect
- Every BOM line has manufacturer, MPN and LCSC fields
- CAN/SPI netclasses defined; power nets removed from SPI class

Co-Authored-By: Claude Opus 5.5 <noreply@anthropic.com>
Parts:
- added C31, C32, C33, C34, C35, C36, C38: 47uF, Capacitor_SMD:C_1206_3216Metric, symbol Device:C
- added C37: 47uF 100V, Capacitor_SMD:CP_Elec_10x10, symbol Device:C_Polarized
- added C39: 1uF, Capacitor_SMD:C_0402_1005Metric, symbol Device:C
- added D4: SS210, Diode_SMD:D_SMA, symbol Diode:SS210
- added D5: SMBJ43A, Diode_SMD:D_SMB, symbol Device:D_Zener
- added F1: 500mA 60V, Fuse:Fuse_1812_4532Metric, symbol Device:Polyfuse
- added R24: 232k, Resistor_SMD:R_0402_1005Metric, symbol Device:R
- added R25, R28: 10k, Resistor_SMD:R_0402_1005Metric, symbol Device:R
- added R27: 33k, Resistor_SMD:R_0402_1005Metric, symbol Device:R
- added U5: TPS2116DRLR, Package_TO_SOT_SMD:SOT-583-8, symbol ebike-controller:TPS2116
- C2, C24: value 0.1uF -> 100nF; LCSC Part Number (none) -> C307331; Manufacturer (none) -> Samsung; Manufacturer Part Number (none) -> CL05B104KB54PNC
- C20, C21: footprint Capacitor_SMD:C_0402_1005Metric -> Capacitor_SMD:C_1210_3225Metric; LCSC Part Number (none) -> C2803397; Manufacturer (none) -> Samsung; Manufacturer Part Number (none) -> CL32Y475KCIVPNE
- C22, C23: footprint Capacitor_SMD:C_0402_1005Metric -> Capacitor_SMD:C_0603_1608Metric; LCSC Part Number (none) -> C15725; Manufacturer (none) -> Samsung; Manufacturer Part Number (none) -> CL10B104KC8NNNC
- C25, C8: LCSC Part Number (none) -> C52923; Manufacturer (none) -> Samsung; Manufacturer Part Number (none) -> CL05A105KA5NQNC
- C26: value 55uF -> 47uF; footprint Capacitor_SMD:C_0402_1005Metric -> Capacitor_SMD:C_1206_3216Metric; LCSC Part Number (none) -> C96123; Manufacturer (none) -> Samsung; Manufacturer Part Number (none) -> CL31A476MPHNNNE
- C3, C4: footprint Capacitor_SMD:C_0402_1005Metric -> Capacitor_SMD:C_0805_2012Metric; LCSC Part Number (none) -> C1779; Manufacturer (none) -> Samsung; Manufacturer Part Number (none) -> CL21A475KAQNNNE
- C5, C6: LCSC Part Number (none) -> C307331; Manufacturer (none) -> Samsung; Manufacturer Part Number (none) -> CL05B104KB54PNC
- C7: value 94uF -> 47uF; footprint Capacitor_SMD:C_0402_1005Metric -> Capacitor_SMD:C_1206_3216Metric; LCSC Part Number (none) -> C96123; Manufacturer (none) -> Samsung; Manufacturer Part Number (none) -> CL31A476MPHNNNE
- L1: Manufacturer (none) -> FAUKU; Manufacturer Part Number (none) -> GSM0630-6R8-M
- L2: value 8.2uH -> 10uH; LCSC Part Number C53462990 -> C53462991; Manufacturer (none) -> JIERR; Manufacturer Part Number (none) -> SRG0630-100-M
- R1, R12: LCSC Part Number (none) -> C25741; Manufacturer (none) -> UNI-ROYAL; Manufacturer Part Number (none) -> 0402WGF1003TCE
- U3, U4: value LM65625SRZTR -> LM65625SRZTRQ1; footprint Jackson:RZT0020A-MFG -> ebike-controller:TI_RZT0020A; symbol Converter_DCDC:LM656x5 -> ebike-controller:LM656x5; LCSC Part Number (none) -> C49305977; Manufacturer (none) -> TI; Manufacturer Part Number (none) -> LM65625SRZTRQ1
Connections:
- net +3V3: now also R1.1, C31.1, C32.1, C33.1
- net +5V: now also C3.2, C4.2, C5.2, C6.2, U3.11 (VIN1), U3.17 (VIN2), U3.7 (EN/UVLO), C38.1, U5.2 (VOUT), U5.7 (VOUT); no longer C26.1, L2.2, U4.20 (BIAS)
- net GND: now also C20.1, C21.1, C22.1, C23.1, C3.1, C4.1, C5.1, C6.1, U3.21 (GND), U4.21 (GND), C31.2, C32.2, C33.2, C34.2, C35.2, C36.2, C37.2, C38.2, C39.2, D5.2 (A), R25.2, R28.2, U5.1 (GND); no longer U3. (GND), U4. (GND)
- net LM656_3V3_VCC: no longer R1.1
- net VCC: now also F1.1; no longer C20.1, C21.1, C22.1, C23.1, C3.1, C4.1, C5.1, C6.1
- net NRST: now reaches R1.2, U3.2 (PG)
- net VIN_PROT: now reaches C20.2, C21.2, C22.2, C23.2, U4.11 (VIN1), U4.17 (VIN2)
- net VIN_PROT: now also C37.1, D4.1 (K), D5.1 (K), R24.1; no longer U4.7 (EN/UVLO)
- new net: D4.2 (A), F1.2
- new net: R27.2, R28.1, U5.4 (PR1)
- new net 5V_BUCK: C26.1, C34.1, C35.1, C36.1, C39.1, L2.2, R27.1, U4.20 (BIAS), U5.3 (VIN1), U5.5 (MODE)
- new net U4_EN: R24.2, R25.1, U4.7 (EN/UVLO)
- new net VBUS: U5.6 (VIN2)
- no-connect marks 0 -> 1
Other:
- note added: "47uF/10V 1206 X5R: ~4x per rail gives >=75uF (3V3) / >=50uF (5V) effective (TI Table 8-1, LM6xx25). C39 1uF: place at U5 VIN1."
- note added: "5V POWER PATH (BUCK PRIORITY, USB FALLBACK)"
- note added: "5V REG UVLO"
- note added: "BATTERY INPUT PROTECTION"
- note added: "EN 1.25V rise / 1.0V fall: on 30.3V, off 24.2V"
- note added: "F1 60V PTC (no nuisance trip on hot-plug inrush), D4 100V reverse-polarity Schottky, D5 SMBJ43A (Vc 69V < 72V abs max), C37 damps cable ringing (TI 8.4)."
- note added: "OUTPUT CAPACITORS (plus C7 / C26 at the regulators)"
- note added: "PR1 = 5V_BUCK x 10k/43k: VIN1 selected above ~4.3V. VBUS only feeds +5V when the buck is off; TPS2116 blocks backfeed into the host."
